Commit message: Adding submodule, updateing shellscript and urdf files

File: catkin_ws/src/easter_egg_hunt/urdf/sick_lm2xx.urdf.xacro (robot description, xacro)
@@ -7,5 +7,5 @@
       <origin xyz="0 0 0" rpy="0 0 ${PI/2}"/>
       <geometry>
-        <mesh filename="package://building_mapper/urdf/meshes/SICK_LM200-LM291_MOUNT.stl" scale="0.001 0.001 0.001"/>
+        <mesh filename="package://easter_egg_hunt/urdf/meshes/SICK_LM200-LM291_MOUNT.stl" scale="0.001 0.001 0.001"/>
       </geometry>
       <material name="black"/>
@@ -24,5 +24,5 @@
       <origin xyz="0 0 0" rpy="0 0 ${PI/2}"/>
       <geometry>
-        <mesh filename="package://building_mapper/urdf/meshes/SICK_LM200-LM291.stl" scale="0.001 0.001 0.001"/>
+        <mesh filename="package://easter_egg_hunt/urdf/meshes/SICK_LM200-LM291.stl" scale="0.001 0.001 0.001"/>
       </geometry>
       <material name="blue"/>
