Commit message: Adding in AR support with almost working transform and calibration.

File: catkin_ws/src/easter_egg_hunt/urdf/loadout.urdf.xacro (robot description, xacro)
@@ -62,3 +62,20 @@
     <material name="blue"/>
   </gazebo>
+  <link name="head_camera">
+    <visual>
+      <origin xyz="0 0 0" rpy="0 0 0"/>
+      <geometry>
+        <cylinder length="0.025" radius="0.01"/>
+      </geometry>
+      <material name="black"/>
+    </visual>
+  </link>
+  <joint name="camera" type="fixed">
+    <parent link="laser"/>
+    <child link="head_camera"/>
+    <origin xyz="0.045 0 0.15" rpy="0 ${PI/2} 0"/>
+  </joint>
+  <gazebo reference="head_camera">
+    <material name="black"/>
+  </gazebo>
 </robot>

Commit message: Updating URDF model to rotate the camera to be the correct orientation.

File: catkin_ws/src/easter_egg_hunt/urdf/loadout.urdf.xacro (robot description, xacro)
@@ -62,5 +62,5 @@
     <material name="blue"/>
   </gazebo>
-  <link name="head_camera">
+  <link name="head_camera_temp">
     <visual>
       <origin xyz="0 0 0" rpy="0 0 0"/>
@@ -71,7 +71,7 @@
     </visual>
   </link>
-  <joint name="camera" type="fixed">
+  <joint name="camera_temp" type="fixed">
     <parent link="laser"/>
-    <child link="head_camera"/>
+    <child link="head_camera_temp"/>
     <origin xyz="0.045 0 0.15" rpy="0 ${PI/2} 0"/>
   </joint>
@@ -79,3 +79,10 @@
     <material name="black"/>
   </gazebo>
+  <link name="head_camera">
+  </link>
+  <joint name="camera" type="fixed">
+    <parent link="head_camera_temp"/>
+    <child link="head_camera"/>
+    <origin xyz="0 0 0" rpy="0 0 ${-PI/2}"/>
+  </joint>
 </robot>
